File: PCB/PCB.kicad_pcb (KiCad board)
At the start: 2 copper layers, 95.2 x 61 mm, 48 parts, among them J1 Conn_01x02, J2 6P4C, J3 Conn_01x03, J4 Conn_02x08_Odd_Even, J5 Conn_01x08, J6 Conn_01x04, J7 Conn_02x03_Odd_Even, U1 LM358, U2 L293D

Commit message: PCB: Update Feather symbol and footprint
This changes from a locally created one to the KiCad library version of
it (which has seen some changes before it was merged).

This also seems to completely rewrite the .kicad_pcb file, so maybe the
earlier conversion to KiCad9 did not work (or was not committed), so
the diff of this commit on the PCB is useless.
Parts:
- removed REF**: KiCad-Logo2_5mm_SilkScreen, Symbol:KiCad-Logo2_5mm_SilkScreen
- A1: value Adafruit Feather M0 -> Adafruit_Feather_M0_Adalogger
- moved A1 21.6 mm to (58.4, 180.3), turned to 90 degrees
- moved C5 1.27 mm to (71.1, 176.5)
- moved R8 1.10 mm to (68.6, 163.7)
- moved R7 1.10 mm to (72.4, 171.3)
Connections:
- A1 pad 1: SDA -> unconnected-(A1-~{RESET}-Pad1)
- A1 pad 10: +5V -> STRIP3
- A1 pad 11: Net-(A1-Pad11) -> STRIP4
- A1 pad 12: Net-(A1-Pad12) -> STRIP5
- A1 pad 13: Net-(A1-Pad13) -> STRIP6
- A1 pad 14: Net-(A1-Pad14) -> STRIP7
- A1 pad 15: Net-(A1-Pad15) -> STRIP8
- A1 pad 17: DAC -> SDA
- A1 pad 18: CURRENT_SENSE -> SCL
- A1 pad 19: Net-(A1-Pad19) -> MOTION
- A1 pad 2: SCL -> unconnected-(A1-3V3-Pad2)
- A1 pad 20: STRIP1 -> BRIDGE_IN_2
- A1 pad 21: STRIP2 -> BRIDGE_IN_1
- A1 pad 22: STRIP3 -> unconnected-(A1-D10-Pad22)
- A1 pad 23: STRIP4 -> unconnected-(A1-D11-Pad23)
- A1 pad 24: STRIP5 -> unconnected-(A1-D12-Pad24)
- A1 pad 25: STRIP6 -> unconnected-(A1-D13-Pad25)
- A1 pad 26: STRIP7 -> +5V
- A1 pad 27: STRIP8 -> unconnected-(A1-EN-Pad27)
- A1 pad 28: GND -> unconnected-(A1-VBAT-Pad28)
- A1 pad 3: MOTION -> unconnected-(A1-AREF-Pad3)
- A1 pad 4: BRIDGE_IN_2 -> GND
- A1 pad 5: BRIDGE_IN_1 -> DAC
- A1 pad 6: Net-(A1-Pad6) -> CURRENT_SENSE
- A1 pad 7: Net-(A1-Pad7) -> unconnected-(A1-A2-Pad7)
- A1 pad 8: Net-(A1-Pad8) -> STRIP1
- A1 pad 9: Net-(A1-Pad9) -> STRIP2
- J2 pad 1: Net-(J2-Pad1) -> unconnected-(J2-Pad1)
- J2 pad 2: Net-(J2-Pad2) -> unconnected-(J2-Pad2)
- J2 pad 5: Net-(J2-Pad5) -> unconnected-(J2-Pad5)
- J2 pad 6: Net-(J2-Pad6) -> unconnected-(J2-Pad6)
- J4 pad 1: Net-(J4-Pad1) -> unconnected-(J4-Pin_1-Pad1)
- J4 pad 10: Net-(J4-Pad10) -> unconnected-(J4-Pin_10-Pad10)
- J4 pad 11: Net-(J4-Pad11) -> unconnected-(J4-Pin_11-Pad11)
- J4 pad 12: Net-(J4-Pad12) -> unconnected-(J4-Pin_12-Pad12)
- J4 pad 13: Net-(J4-Pad13) -> unconnected-(J4-Pin_13-Pad13)
- J4 pad 14: Net-(J4-Pad14) -> unconnected-(J4-Pin_14-Pad14)
- J4 pad 15: Net-(J4-Pad15) -> unconnected-(J4-Pin_15-Pad15)
- J4 pad 16: Net-(J4-Pad16) -> unconnected-(J4-Pin_16-Pad16)
- J4 pad 2: Net-(J4-Pad2) -> unconnected-(J4-Pin_2-Pad2)
- J4 pad 3: Net-(J4-Pad3) -> unconnected-(J4-Pin_3-Pad3)
- J4 pad 4: Net-(J4-Pad4) -> unconnected-(J4-Pin_4-Pad4)
- J4 pad 5: Net-(J4-Pad5) -> unconnected-(J4-Pin_5-Pad5)
- J4 pad 6: Net-(J4-Pad6) -> unconnected-(J4-Pin_6-Pad6)
- J4 pad 7: Net-(J4-Pad7) -> unconnected-(J4-Pin_7-Pad7)
- J4 pad 8: Net-(J4-Pad8) -> unconnected-(J4-Pin_8-Pad8)
- J4 pad 9: Net-(J4-Pad9) -> unconnected-(J4-Pin_9-Pad9)
- RV1 pad 3: Net-(RV1-Pad3) -> unconnected-(RV1-Pad3)
- U2 pad 11: Net-(U2-Pad11) -> unconnected-(U2-3Y-Pad11)
- U2 pad 14: Net-(U2-Pad14) -> unconnected-(U2-4Y-Pad14)
Routing:
- net +5V: track 198.5 -> 170.4 mm
- net Net-(U1B--): track 19.1 -> 20.2 mm
- net CURRENT_SENSE: track 23.3 -> 22.2 mm
- net BRIDGE_IN_1: track 38.6 -> 39.6 mm
- net MOTION: track 24.1 -> 25.0 mm, vias 0 -> 1
- net BRIDGE_IN_2: track 22.5 -> 23.3 mm, vias 0 -> 1
- net unconnected-(A1-~{RESET}-Pad1): vias 0 -> 2
- net unconnected-(A1-D13-Pad25): vias 0 -> 1
- net STRIP8: vias 0 -> 2
- net STRIP3: vias 0 -> 1
- net SCL: vias 0 -> 1
- net GND: vias 111 -> 102
Other:
- net class Default removed
- net class Power removed
- net class Telephone removed

Commit message: PCB: Update all symbols from library
Parts:
- U2: footprint Package_DIP:DIP-16_W7.62mm_Socket_LongPads -> Package_DIP:DIP-16_W7.62mm
